Commit message: 修复多次导航后机器人卡死的问题

File: src/gazebo_modele/urdf/model.urdf (robot description, URDF)
Before this commit: robot lio, 9 links, 8 joints
Links:
- added link rear_caster_link, mass 0.08; collision sphere radius=0.024; visual sphere radius=0.024
- link base_link: mass 0.1 -> 6.0; geometry collision cylinder length=0.08 radius=0.11; visual cylinder length=0.08 radius=0.12
- link caster_link: mass 0.02 -> 0.08; geometry collision sphere radius=0.024; visual sphere radius=0.024
- link gps_link: mass 0.1 -> 0.05
- link imu_link: mass 0.1 -> 0.05; geometry collision box size=0.025 0.025 0.015; visual box size=0.025 0.025 0.015
- link left_wheel_link: mass 0.2 -> 0.5; geometry collision cylinder length=0.03 radius=0.055; visual cylinder length=0.03 radius=0.055
- link navsat_link: mass 0.1 -> 0.05
- link right_wheel_link: mass 0.2 -> 0.5; geometry collision cylinder length=0.03 radius=0.055; visual cylinder length=0.03 radius=0.055
- link velodyne: mass 0.1 -> 0.15; geometry collision cylinder length=0.04 radius=0.035; visual cylinder length=0.04 radius=0.035
Joints:
- added joint rear_caster_joint: type fixed, parent base_link, child rear_caster_link, origin xyz=-0.105 0.0 -0.031 rpy=0 0 0
- joint base_joint: origin xyz=0.0 0.0 0.36 rpy=0 0 0 -> xyz=0 0 0.055 rpy=0 0 0
- joint caster_joint: axis 0 1 0 -> (none); origin xyz=0.06 0.0 -0.041 -> xyz=0.105 0.0 -0.031 rpy=0 0 0
- joint gps_joint: origin xyz=-0.1 0 0.1 -> xyz=0.09 -0.06 0.10 rpy=0 0 0
- joint imu_joint: origin xyz=0 0 0.02 -> xyz=0 0 0.095 rpy=0 0 0
- joint left_wheel_joint: origin xyz=-0.04 0.10 -0.04 -> xyz=0.02 0.115 0.0 rpy=0 0 0
- joint lidar_joint: origin xyz=0 0 0.02 -> xyz=0.08 0 0.105 rpy=0 0 0
- joint navsat_joint: origin xyz=0.1 0 0.1 -> xyz=0.09 0.06 0.10 rpy=0 0 0
- joint right_wheel_joint: origin xyz=-0.04 -0.10 -0.04 -> xyz=0.02 -0.115 0.0 rpy=0 0 0

Commit message: 更新定位

File: src/gazebo_modele/urdf/model.urdf (robot description, URDF)
Before this commit: robot fishbot, 10 links, 9 joints
Links:
- added link camera_link, mass 0.05; collision box size=0.03 0.03 0.02; visual box size=0.03 0.03 0.02
- added link camera_optical_frame
Joints:
- added joint camera_joint: type fixed, parent base_link, child camera_link, origin xyz=0.10 0.0 0.11 rpy=0 0 0
- added joint camera_optical_joint: type fixed, parent camera_link, child camera_optical_frame, origin xyz=0 0 0 rpy=-1.57079632679 0 -1.57079632679

Commit message: 加回视觉里程计增益

File: src/gazebo_modele/urdf/model.urdf (robot description, URDF)
Before this commit: robot fishbot, 12 links, 11 joints
Joints:
- joint caster_joint: axis (none) -> 0 0 1; type fixed -> continuous
- joint rear_caster_joint: axis (none) -> 0 0 1; type fixed -> continuous

Commit message: 修改轮子碰撞模型为球体

File: src/gazebo_modele/urdf/model.urdf (robot description, URDF)
Before this commit: robot fishbot, 12 links, 11 joints
Links:
- link left_wheel_link: geometry collision sphere radius=0.055; visual cylinder length=0.03 radius=0.055
- link right_wheel_link: geometry collision sphere radius=0.055; visual cylinder length=0.03 radius=0.055
